File: v5/air-quality-pcb-v5.kicad_sch (KiCad schematic)
At the start: 65 parts, among them J1 USB-C, J3 SERVO, J4 LiPo, J5 SPARE, Q1 MMBT2222A, Q2 MMBT2222A, Q3 DMG2305UX, Q4 DMG2305UX, SW1 RESET, SW2 BOOT, SW3 POWER, U1 ESP-12F, U2 CP2102N-A02-GQFN28, U3 MCP73831, U4 AP2112K-3.3, U5 BME688, U6 USBLC6-2SC6, U7 MT3608

Commit message: Update v5 add bom
Parts:
- C1, C12, C14, C15, C17, C3, C5, C8: MPN (none) -> CL21B104KBCNNNC; Manufacturer (none) -> Samsung Electro-Mechanics
- C10: MPN (none) -> CL21B105KOFNNWE; Manufacturer (none) -> Samsung Electro-Mechanics
- C11, C16, C18, C2: MPN (none) -> CC0805KRX5R7BB106; Manufacturer (none) -> YAGEO
- C13: MPN (none) -> UCD1C101MCL1GS; Manufacturer (none) -> Nichicon
- C19: MPN (none) -> CL21A226KOQNNNG; Manufacturer (none) -> Samsung Electro-Mechanics
- C4, C6, C7, C9: MPN (none) -> CL21A475KOFNNNG; Manufacturer (none) -> Samsung Electro-Mechanics
- D1: MPN (none) -> B5819W-TP; Manufacturer (none) -> MCC (Micro Commercial Components)
- D2: MPN (none) -> LTST-C170GKT; Manufacturer (none) -> Lite-On Inc.
- D3: MPN (none) -> LTST-C170TBKT; Manufacturer (none) -> Lite-On Inc.
- D4: MPN (none) -> SS34-HF; Manufacturer (none) -> Comchip Technology
- J1: MPN (none) -> TYPE-C-31-M-12; Manufacturer (none) -> Korean Hroparts (HRO)
- J3: MPN (none) -> 61300311121; Manufacturer (none) -> Wurth Elektronik
- J4: MPN (none) -> B2B-PH-K-S; Manufacturer (none) -> JST
- J5: MPN (none) -> 61300411121; Manufacturer (none) -> Wurth Elektronik
- L1: MPN (none) -> SWPA4030S100MT; Manufacturer (none) -> Sunlord
- Q1, Q2: MPN (none) -> MMBT2222ALT1G; Manufacturer (none) -> onsemi
- Q3, Q4: MPN (none) -> DMG2305UX-7; Manufacturer (none) -> Diodes Incorporated
- R1, R18, R19, R2, R3, R4, R5, R6, R7: MPN (none) -> RC0805FR-0710KL; Manufacturer (none) -> YAGEO
- R10, R11: MPN (none) -> RC0805FR-075K1L; Manufacturer (none) -> YAGEO
- R12: MPN (none) -> RC0805FR-0722K1L; Manufacturer (none) -> YAGEO
- R13: MPN (none) -> RC0805FR-0747K5L; Manufacturer (none) -> YAGEO
- R14: MPN (none) -> RC0805FR-072K2L; Manufacturer (none) -> YAGEO
- R15, R16: MPN (none) -> RC0805FR-071KL; Manufacturer (none) -> YAGEO
- R17: MPN (none) -> RC0805FR-07100RL; Manufacturer (none) -> YAGEO
- R20, R9: MPN (none) -> RC0805FR-07100KL; Manufacturer (none) -> YAGEO
- R21: MPN (none) -> RC0805FR-0727KL; Manufacturer (none) -> YAGEO
- R22: MPN (none) -> RC0805FR-0782KL; Manufacturer (none) -> YAGEO
- R23: MPN (none) -> RC0805FR-0711KL; Manufacturer (none) -> YAGEO
- SW1, SW2: MPN (none) -> KMR221G LFS; Manufacturer (none) -> C&K
- SW3: MPN (none) -> PCM12SMTBR; Manufacturer (none) -> C&K
- U1: MPN (none) -> ESP-12F; Manufacturer (none) -> Ai-Thinker
- U2: MPN (none) -> CP2102N-A02-GQFN28; Manufacturer (none) -> Silicon Labs
- U3: MPN (none) -> MCP73831T-2ACI/OT; Manufacturer (none) -> Microchip Technology
- U4: MPN (none) -> AP2112K-3.3TRG1; Manufacturer (none) -> Diodes Incorporated
- U5: MPN (none) -> BME688; Manufacturer (none) -> Bosch Sensortec
- U6: MPN (none) -> USBLC6-2SC6; Manufacturer (none) -> STMicroelectronics
- U7: MPN (none) -> MT3608; Manufacturer (none) -> Aerosemi Tech
