File: v5/air-quality-pcb-v5.kicad_pcb (KiCad board)
At the start: 2 copper layers, 72 x 72 mm, 74 parts, among them J1 USB-C, J3 SERVO, J4 LiPo, J5 SPARE, Q1 MMBT2222A, Q2 MMBT2222A, Q3 DMG2305UX, Q4 DMG2305UX, SW1 RESET, SW2 BOOT, SW3 POWER, U1 ESP-12F, U2 CP2102N-A02-GQFN28, U3 MCP73831, U4 AP2112K-3.3, U5 BME688, U6 USBLC6-2SC6, U7 MT3608

Commit message: Update v5
Parts:
- removed the Q4 at (30.5, 50.0)
- removed the R22 at (74.5, 56.0)
- moved R2 39.8 mm to (42.5, 34.0), turned to -90 degrees
- moved C3 38.9 mm to (56.5, 33.0), turned to 180 degrees
- moved C11 32.1 mm to (60.5, 35.5)
- moved C2 31.7 mm to (60.5, 33.0)
- moved C13 31.2 mm to (85.0, 59.5), turned to -90 degrees
- moved R5 30.1 mm to (66.8, 55.7), turned to -90 degrees
- moved C5 29.5 mm to (37.0, 80.0), turned to 180 degrees
- moved C4 29.0 mm to (37.0, 82.0), turned to 180 degrees
- moved R1 25.6 mm to (60.5, 30.5)
- moved C12 25.0 mm to (56.5, 35.5), turned to 180 degrees
- moved R9 24.9 mm to (36.5, 53.0)
- moved C6 24.5 mm to (36.5, 51.0)
- moved R16 23.9 mm to (70.5, 56.5), turned to -90 degrees
- moved R21 23.9 mm to (38.5, 58.5), turned to 180 degrees
- moved C1 23.4 mm to (56.5, 30.5), turned to 180 degrees
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Routing:
- net /GND: track 387.0 -> 0.00 mm, vias 4 -> 0
- net /VBAT: track 97.7 -> 54.6 mm
- net /CP_VDD: track 43.9 -> 4.62 mm, vias 2 -> 0
- net /+3V3: track 175.5 -> 140.1 mm, vias 4 -> 2
- net /RST: track 94.0 -> 59.2 mm, vias 2 -> 3
- net /GPIO2: track 39.2 -> 8.13 mm, vias 2 -> 0
- net /SCL: track 39.3 -> 66.1 mm
- net /SERVO_PWM: track 26.3 -> 0.00 mm
- net /LED_STAT: track 28.3 -> 2.43 mm, vias 2 -> 0
- net /SDA: track 46.3 -> 68.0 mm
- net /PROG: track 24.4 -> 3.42 mm, vias 2 -> 0
- net /CC2: track 23.3 -> 3.65 mm, vias 2 -> 0
- net /VBAT_SENSE: track 37.7 -> 21.2 mm, vias 2 -> 4
- net /GPIO12: track 46.4 -> 30.8 mm, vias 0 -> 1
- net /BOOST_FB: track 22.8 -> 7.23 mm
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- added copper zone on B.Cu, net /GND
- added copper zone on F.Cu, net /GND
- removed copper zone on B.Cu, net GND
- removed copper zone on F.Cu, net GND

Commit message: Update v5 add bom
Routing:
- net /GND: track 0.00 -> 96.8 mm, vias 0 -> 12
- net /SERVO_PWM: track 0.00 -> 30.2 mm, vias 0 -> 2

Commit message: Update vias
Routing:
- net /GND: track 96.8 -> 107.2 mm, vias 12 -> 13
- net /VBAT_SENSE: track 21.2 -> 30.5 mm
- net /SDA: track 68.0 -> 73.7 mm
- net /RST: track 59.2 -> 64.8 mm
- net /SCL: track 66.1 -> 70.6 mm
- net /UART_RX: track 37.3 -> 39.1 mm
- net /GPIO0: track 47.8 -> 49.4 mm
- net /UART_TX: track 38.0 -> 38.6 mm
- net /BAT_IN: vias 1 -> 0
