File: v6/air-quality-pcb-v6.kicad_sch (KiCad schematic)
At the start: 65 parts, among them J1 USB-C, J3 SERVO, J4 LiPo, Q1 MMBT2222A, Q2 MMBT2222A, Q3 DMG2305UX, Q4 DMG2305UX, SW1 RESET, SW2 BOOT, SW3 POWER, SW4 WIFI_MODE, U1 ESP-12F, U2 CP2102N-A02-GQFN28, U3 MCP73831, U4 AP2112K-3.3, U5 BME688, U6 USBLC6-2SC6, U7 MT3608

Commit message: Update
Other:
- note added: "WiFi Mode Switch (SW4) POS.1 = OFF (GPIO12 low) POS.2 = SPARSE, upload 1x/h (both inputs high) POS.3 = CONTINUOUS (GPIO14 low). Read at boot with internal pull-ups (no external pull-ups: +3V3 stays live in deep sleep)."
- note removed: "WiFi Mode Switch (SW4): POS.1 = OFF (GPIO12 low) — POS.2 = SPARSE, upload 1x/h (both inputs high) — POS.3 = CONTINUOUS (GPIO14 low). Read at boot with internal pull-ups (no external pull-ups: +3V3 stays live in deep sleep)."
Changed lines of the file:
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@@
 		)
 	)
-	(text "WiFi Mode Switch (SW4): POS.1 = OFF (GPIO12 low) — POS.2 = SPARSE, upload 1x/h (both inputs high) — POS.3 = CONTINUOUS (GPIO14 low). Read at boot with internal pull-ups (no external pull-ups: +3V3 stays live in deep sleep)."
+	(text "WiFi Mode Switch (SW4)\nPOS.1 = OFF (GPIO12 low)\nPOS.2 = SPARSE, upload 1x/h (both inputs high)\nPOS.3 = CONTINUOUS (GPIO14 low).\nRead at boot with internal pull-ups\n(no external pull-ups: +3V3 stays live in deep sleep)."
 		(exclude_from_sim no)
-		(at 60 276 0)
+		(at 118.11 72.644 0)
 		(effects
 			(font
-				(size 1.5 1.5)
+				(size 0.508 0.508)
 			)
 			(justify left bottom)
