File: v7/air-quality-pcb-v7.kicad_pcb (KiCad board)
At the start: 2 copper layers, 72 x 62.2 mm, 85 parts, among them J1 USB-C, J3 SERVO, J4 LiPo, J5 STEMMA_QT, Q10 BSS138, Q3 DMG2305UX, Q4 DMG2305UX, Q5 DMG2305UX, Q6 DMG2305UX, Q7 2N7002, Q8 DMG2305UX, Q9 BSS138, SW1 RESET, SW2 BOOT, SW3 POWER, SW4 WIFI_MODE, U1 ESP32-C3-WROOM-02, U3 MCP73831, U4 AP2112K-3.3, U5 BME688, U6 USBLC6-2SC6, U7 MT3608, U8 USBLC6-2SC6

Commit message: Add v9
Parts:
- SW4: footprint AirQuality:SW_Slide_SP3T_Angled_CK_OS103011MA7Q -> SamacSys_Parts:OS103011MA7QP1
- U1: footprint AirQuality:ESP32-C3-WROOM-02_EPADvia0.3 -> RF_Module:ESP32-C3-WROOM-02
