File: v9/air-quality-pcb-v9.kicad_sch (KiCad schematic)
At the start: 78 parts, among them J1 USB-C, J3 SERVO, J4 LiPo, J5 STEMMA_QT, Q10 BSS138, Q3 DMG2305UX, Q4 DMG2305UX, Q5 DMG2305UX, Q6 DMG2305UX, Q7 2N7002, Q8 DMG2305UX, Q9 BSS138, SW1 RESET, SW2 BOOT, SW3 POWER, SW4 WIFI_MODE, U1 ESP32-C3-WROOM-02, U3 MCP73831, U4 AP2112K-3.3, U5 BME688, U6 USBLC6-2SC6, U7 MT3608, U8 USBLC6-2SC6

Commit message: Add v9
Parts:
- removed C18, C21: 22uF, Capacitor_SMD:C_0805_2012Metric, symbol Device:C
- removed D4: PMEG4030ER, Diode_SMD:Nexperia_CFP3_SOD-123W, symbol Device:D_Schottky
- removed L1: 10uH, Inductor_SMD:L_Sunlord_SWPA4030S, symbol Device:L
- removed R22: 82k, Resistor_SMD:R_0805_2012Metric, symbol Device:R
- removed R23: 11k, Resistor_SMD:R_0805_2012Metric, symbol Device:R
- removed U7: MT3608, Package_TO_SOT_SMD:SOT-23-6, symbol Regulator_Switching:MT3608
- added C24: 100nF, Capacitor_SMD:C_0805_2012Metric, symbol Device:C
- U1: footprint RF_Module:ESP32-C3-WROOM-02 -> Espressif:ESP32-C3-WROOM-02
Connections:
- net SERVO_5V is gone; now on net SERVO_PWR: C13.1, C19.1, J3.2 (Pin_2)
- net GND: now also C24.2
- net MODE_A: now also U1.3 (IO4); no longer U1.15 (IO3)
- net MODE_B: now also U1.4 (IO5); no longer U1.3 (IO4)
- net QT_3V3: now also C24.1
- net SERVO_PWM: now also U1.18 (IO0); no longer U1.4 (IO5)
- net USB_D+: now also U6.1 (I/O1); no longer U6.6 (I/O1)
- net USB_D-: now also U6.3 (I/O2); no longer U6.4 (I/O2)
- net USB_DM_CON: now also U6.4 (I/O2); no longer U6.3 (I/O2)
- net USB_DP_CON: now also U6.6 (I/O1); no longer U6.1 (I/O1)
- net VBAT_SENSE: now also U1.15 (IO3); no longer U1.18 (IO0)
- net BOOST_EN renamed SERVO_EN
- net BOOST_GATE renamed SERVO_GATE
- net BOOST_IN renamed SERVO_PWR
- net BOOST_PD renamed SERVO_PD
- no-connect marks 6 -> 5
Other:
- note added: "ESP32-C3 notes (MCU box): Strapping: IO2 (R2), IO8 (R5), IO9 (R3) pulled up 10k -> SPI boot. BOOT (SW2) low at reset -> USB download mode. IO8 drives the STATUS LED active-low (LED off = strap high). IO10 = SERVO_EN; R4 100k keeps the servo rail off at reset/sleep. EN: R1 10k + C1 1uF RC delay (Espressif HW design guide). USB: IO18/IO19 native USB Serial/JTAG - no UART bridge. SW4 (OS103011MA7QP1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"
- note added: "Servo Rail Load Switch"
- note added: "Servo rail load switch (v8: no boost, the servo runs from VSYS = USB via D1 ~4.5 V or the battery 3.0-4.2 V). Q6 connects SERVO_PWR to VSYS only while SERVO_EN (IO10) is high. Q7 pulls the gate to ~VSYS-2.5 V via R28; R4 keeps it off at reset/sleep. C22 (gate-drain) slews SERVO_PWR at ~0.5 V/ms -> ~60 mA inrush into C13 + C19 (122 uF). Firmware: SERVO_EN high >= 50 ms before a move; skip moves be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"
- note removed: "ESP32-C3 notes (MCU box): Strapping: IO2 (R2), IO8 (R5), IO9 (R3) pulled up 10k -> SPI boot. BOOT (SW2) low at reset -> USB download mode. IO8 drives the STATUS LED active-low (LED off = strap high). IO10 = BOOST_EN; R4 100k keeps the boost off at reset/sleep. EN: R1 10k + C1 1uF RC delay (Espressif HW design guide). USB: IO18/IO19 native USB Serial/JTAG - no UART bridge. SW4 (OS103011MA7QP1, com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"
- note removed: "Layout: hot loop U7 SW -> D4 -> C19/C21 -> GND -> U7 pin 2 within ~8x8 mm on F.Cu. C18 (22 uF) at U7 pin 5, L1 at pin 1, R22/R23 at pin 3. No signals under L1 / the SW node."
- note removed: "Servo 5V Boost (MT3608)"
- note removed: "Servo rail load switch (v7). A boost converter is not off when EN is low: VSYS -> L1 -> D4 still feeds SERVO_5V (servo idle + R22/R23). Q6 disconnects BOOST_IN from VSYS while BOOST_EN (IO10) is low. Q7 pulls the gate to ~VSYS-2.5 V via R28 when BOOST_EN is high. C22 (gate-drain) slews BOOST_IN at ~0.5 V/ms -> ~80 mA inrush into ~166 uF downstream. Firmware: BOOST_EN high >= 100 ms before a move."
